File: power.kicad_sch (KiCad schematic)
At the start: 6 parts, among them J4 10103592-0001LF, U2 AMS1117-3.3

Commit message: base mcu decoupling cap routing
Parts:
- J4: footprint USB:AMPHENOL_10103592-0001LF -> 10103592-0001LF:AMPHENOL_10103592-0001LF
Changed lines of the file:
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@@
 			)
 		)
-		(property "Footprint" "USB:AMPHENOL_10103592-0001LF"
+		(property "Footprint" "10103592-0001LF:AMPHENOL_10103592-0001LF"
 			(at 83.82 73.66 0)
 			(effects
