File: _autosave-microcontroller.kicad_sch (KiCad schematic)
At the start: 16 parts, among them SW1 System Reset, SW2 Boot Switch, U1 STM32F446RETx

Commit message: fix power supply scheme for microcontroller schematic
Changed lines of the file:
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@@
 	(text "Power Supply Scheme"
 		(exclude_from_sim no)
-		(at 70.866 19.304 0)
+		(at 54.864 19.558 0)
 		(effects
 			(font
