File: microcontroller.kicad_sch (KiCad schematic)
At the start: 16 parts, among them SW1 System Reset, SW2 Boot Switch, U1 STM32F446RETx

Commit message: replace usb interface with usb-c. add data lines for it too
Connections:
- net USB_OTG_FS_DM: now reaches U1.44 (PA11)
- net USB_OTG_FS_DP: now reaches U1.45 (PA12)
- no-connect marks 35 -> 33
Other:
- note added: "USB"
Changed lines of the file:
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@@
+	)
+	(rectangle
+		(start 200.66 102.235)
+		(end 222.25 108.585)
+		(stroke
+			(width 0)
+			(type default)
+		)
+		(fill
+			(type none)
+		)
 	)
 	(rectangle
@@
 		)
 	)
-	(text "AN4488 Page 26"
-		(exclude_from_sim no)
-		(at 52.832 101.6 0)
-		(effects
-			(font
-				(size 1.27 1.27)
-				(italic yes)
-			)
-		)
-	)
-	(text "Boot Mode"
-		(exclude_from_sim no)
-		(at 37.084 76.962 0)
+	(text "USB"
+		(exclude_from_sim no)
+		(at 217.678 101.092 0)
 		(effects
 			(font
@@
 		)
 	)
-	(text "SPI1 Bus"
-		(exclude_from_sim no)
-		(at 210.185 85.725 0)
+	(text "AN4488 Page 26"
+		(exclude_from_sim no)
+		(at 52.832 101.6 0)
+		(effects
+			(font
+				(size 1.27 1.27)
+				(italic yes)
+			)
+		)
+	)
+	(text "Boot Mode"
+		(exclude_from_sim no)
+		(at 37.084 76.962 0)
 		(effects
 			(font
@@
 		)
 	)
-	(text "AN4488 Page 9\n"
-		(exclude_from_sim no)
-		(at 87.884 49.022 0)
-		(effects
-			(font
-				(size 1.27 1.27)
-				(italic yes)
-			)
-		)
-	)
-	(text "Servo GPIO"
-		(exclude_from_sim no)
-		(at 208.788 73.152 0)
+	(text "SPI1 Bus"
+		(exclude_from_sim no)
+		(at 210.185 85.725 0)
 		(effects
 			(font
@@
 		)
 	)
-	(text "Pull to ground to \nenter reset state"
-		(exclude_from_sim no)
-		(at 40.132 67.056 0)
-		(effects
-			(font
-				(size 1.27 1.27)
-			)
-			(justify left)
-		)
-	)
-	(text "System Reset"
-		(exclude_from_sim no)
-		(at 37.592 44.45 0)
+	(text "AN4488 Page 9\n"
+		(exclude_from_sim no)
+		(at 87.884 49.022 0)
+		(effects
+			(font
+				(size 1.27 1.27)
+				(italic yes)
+			)
+		)
+	)
+	(text "Servo GPIO"
+		(exclude_from_sim no)
+		(at 208.788 73.152 0)
 		(effects
 			(font
@@
 		)
 	)
-	(text "Power Supply Scheme"
-		(exclude_from_sim no)
-		(at 77.724 23.368 0)
+	(text "Pull to ground to \nenter reset state"
+		(exclude_from_sim no)
+		(at 40.132 67.056 0)
+		(effects
+			(font
+				(size 1.27 1.27)
+			)
+			(justify left)
+		)
+	)
+	(text "System Reset"
+		(exclude_from_sim no)
+		(at 37.592 44.45 0)
 		(effects
 			(font
@@
 		)
 	)
-	(text "VBAT to VDD if no backup battery"
-		(exclude_from_sim no)
-		(at 96.52 46.99 0)
-		(effects
-			(font
-				(size 1.27 1.27)
-			)
-		)
-	)
-	(text "1 - Boot from main flash"
-		(exclude_from_sim no)
-		(at 41.656 80.01 0)
-		(effects
-			(font
-				(size 1.27 1.27)
-			)
-			(justify left)
-		)
-	)
-	(text "VDD bulk capacitor"
-		(exclude_from_sim no)
-		(at 104.648 30.48 0)
-		(effects
-			(font
-				(size 1.27 1.27)
-			)
-		)
-	)
-	(text "VDDA decoupling capacitors"
-		(exclude_from_sim no)
-		(at 182.372 29.21 0)
-		(effects
-			(font
-				(size 1.27 1.27)
-			)
-		)
-	)
-	(text "VCAP"
-		(exclude_from_sim no)
-		(at 75.438 138.43 0)
+	(text "Power Supply Scheme"
+		(exclude_from_sim no)
+		(at 77.724 23.368 0)
 		(effects
 			(font
@@
 		)
 	)
-	(text "USART1 Bus"
-		(exclude_from_sim no)
-		(at 202.692 125.222 0)
+	(text "VBAT to VDD if no backup battery"
+		(exclude_from_sim no)
+		(at 96.52 46.99 0)
+		(effects
+			(font
+				(size 1.27 1.27)
+			)
+		)
+	)
+	(text "1 - Boot from main flash"
+		(exclude_from_sim no)
+		(at 41.656 80.01 0)
+		(effects
+			(font
+				(size 1.27 1.27)
+			)
+			(justify left)
+		)
+	)
+	(text "VDD bulk capacitor"
+		(exclude_from_sim no)
+		(at 104.648 30.48 0)
+		(effects
+			(font
+				(size 1.27 1.27)
+			)
+		)
+	)
+	(text "VDDA decoupling capacitors"
+		(exclude_from_sim no)
+		(at 182.372 29.21 0)
+		(effects
+			(font
+				(size 1.27 1.27)
+			)
+		)
+	)
+	(text "VCAP"
+		(exclude_from_sim no)
+		(at 75.438 138.43 0)
 		(effects
 			(font
@@
 		)
 	)
-	(text "I2C1 Bus"
-		(exclude_from_sim no)
-		(at 203.454 139.192 0)
+	(text "USART1 Bus"
+		(exclude_from_sim no)
+		(at 202.692 125.222 0)
 		(effects
 			(font
@@
 		)
 	)
-	(text "Programming"
-		(exclude_from_sim no)
-		(at 208.28 111.76 0)
+	(text "I2C1 Bus"
+		(exclude_from_sim no)
+		(at 203.454 139.192 0)
 		(effects
 			(font
@@
 		)
 	)
+	(text "Programming"
+		(exclude_from_sim no)
+		(at 208.28 111.76 0)
+		(effects
+			(font
+				(size 1.27 1.27)
+				(thickness 0.254)
+				(bold yes)
+			)
+			(justify left)
+		)
+	)
 	(junction
 		(at 119.38 44.45)
@@
 	)
 	(no_connect
-		(at 168.91 104.14)
-	)
-	(no_connect
 		(at 128.27 88.9)
 	)
@@
 	)
 	(no_connect
-		(at 168.91 106.68)
-	)
-	(no_connect
 		(at 168.91 127)
 	)
@@
 	(wire
 		(pts
+			(xy 168.91 106.68) (xy 203.2 106.68)
+		)
+		(stroke
+			(width 0)
+			(type default)
+		)
+	)
+	(wire
+		(pts
 			(xy 193.04 146.05) (xy 203.2 146.05)
 		)
@@
 		(pts
 			(xy 123.19 111.76) (xy 101.6 111.76)
+		)
+		(stroke
+			(width 0)
+			(type default)
+		)
+	)
+	(wire
+		(pts
+			(xy 168.91 104.14) (xy 203.2 104.14)
 		)
 		(stroke
@@
 		)
 	)
+	(hierarchical_label "USB_OTG_FS_DP"
+		(shape bidirectional)
+		(at 203.2 106.68 0)
+		(effects
+			(font
+				(size 1.27 1.27)
+			)
+			(justify left)
+		)
+	)
 	(hierarchical_label "SERVO_FEEDBACK"
 		(shape input)
@@
 		(effects
 			(font
+				(size 1.27 1.27)
+			)
+			(justify left)
+		)
+	)
+	(hierarchical_label "USB_OTG_FS_DM"
+		(shape bidirectional)
+		(at 203.2 104.14 0)
+		(effects
+			(font
